Commit message: add intial

File: resources/robots/XBot/urdf/fudan_humanoid.urdf (robot description, URDF)
Before this commit: robot fudan_humanoid, 15 links, 14 joints
Links:
- link right_leg_pitch_link: mass 0 -> 0.5141

Commit message: first vision

File: resources/robots/XBot/urdf/fudan_humanoid.urdf (robot description, URDF)
Before this commit: robot fudan_humanoid, 15 links, 14 joints
Links:
- link L_foot: mass 0.583662375025109 -> 0.58366
- link R_foot: mass 0.583662375025108 -> 0.58366
- link base_link: mass 27.458 -> 27.766
- link left_ankle_pitch_link: mass 0.121110895209696 -> 0.10749; geometry visual mesh filename=../meshes/left_ankle_pitch_link.STL
- link left_ankle_roll_link: mass 0.211279168543597 -> 0.14038; geometry visual mesh filename=../meshes/left_ankle_roll_link.STL
- link left_knee_link: mass 2.73838325446566 -> 2.7384; geometry visual mesh filename=../meshes/left_knee_link.STL
- link left_leg_pitch_link: mass 1.53497057709751 -> 1.535; geometry visual mesh filename=../meshes/left_leg_pitch_link.STL
- link left_leg_roll_link: mass 1.1585681644247 -> 1.0891; geometry visual mesh filename=../meshes/left_leg_roll_link.STL
- link left_leg_yaw_link: mass 3.6405005153043 -> 3.6405; geometry visual mesh filename=../meshes/left_leg_yaw_link.STL
- link right_ankle_pitch_link: mass 0.121110895209696 -> 0.10749; geometry visual mesh filename=../meshes/right_ankle_pitch_link.STL
- link right_ankle_roll_link: mass 0.211279168543596 -> 0.14038; geometry visual mesh filename=../meshes/right_ankle_roll_link.STL
- link right_knee_link: mass 2.7383889302029 -> 2.7384; geometry visual mesh filename=../meshes/right_knee_link.STL
- link right_leg_pitch_link: mass 0.5141 -> 1.6695; geometry visual mesh filename=../meshes/right_leg_pitch_link.STL
- link right_leg_roll_link: mass 1.1585681644247 -> 1.0891; geometry visual mesh filename=../meshes/right_leg_roll_link.STL
- link right_leg_yaw_link: mass 3.6407780899498 -> 3.6408; geometry visual mesh filename=../meshes/right_leg_yaw_link.STL
Joints:
- joint left_ankle_pitch_joint: origin xyz=0.015 0.000700000000000006 -0.37 rpy=0 0 0 -> xyz=0.015 0.0007 -0.37 rpy=0 0 0
- joint left_knee_joint: origin xyz=0 0.0199999999998428 -0.4151 rpy=0 0 0 -> xyz=0 0.02 -0.4151 rpy=0 0 0
- joint left_leg_yaw_joint: origin xyz=-0.0579000000000937 0 0.0351 rpy=0 0 0 -> xyz=-0.0579 0 0.0351 rpy=0 0 0
- joint right_ankle_pitch_joint: origin xyz=0.015 -0.000700000000000006 -0.37 rpy=0 0 0 -> xyz=0.015 -0.0007 -0.37 rpy=0 0 0
- joint right_knee_joint: origin xyz=0 -0.0199999999998428 -0.4151 rpy=0 0 0 -> xyz=0 -0.02 -0.4151 rpy=0 0 0
- joint right_leg_pitch_joint: axis 0 0.866025403784429 0.500000000000017 -> 0 0.86603 0.5; origin xyz=0 -0.0264884942777566 -0.116000000000002 rpy=0 0 0 -> xyz=0 -0.026488 -0.116 rpy=0 0 0
- joint right_leg_roll_joint: origin xyz=0.0579 -0.119511505722243 -0.0689999999999984 rpy=0 0 0 -> xyz=0.0579 -0.11951 -0.069 rpy=0 0 0
- joint right_leg_yaw_joint: origin xyz=-0.0578999999999063 0 0.0351 rpy=0 0 0 -> xyz=-0.0579 0 0.0351 rpy=0 0 0

Commit message: add cylinder collision for leg

File: resources/robots/XBot/urdf/fudan_humanoid.urdf (robot description, URDF)
Before this commit: robot fudan_humanoid, 15 links, 14 joints
Links:
- link left_knee_link: geometry collision cylinder length=0.28 radius=0.03; visual mesh filename=../meshes/left_knee_link.STL
- link left_leg_yaw_link: geometry collision cylinder length=0.30 radius=0.04; visual mesh filename=../meshes/left_leg_yaw_link.STL
- link right_knee_link: geometry collision cylinder length=0.28 radius=0.03; visual mesh filename=../meshes/right_knee_link.STL
- link right_leg_yaw_link: geometry collision cylinder length=0.30 radius=0.04; visual mesh filename=../meshes/right_leg_yaw_link.STL
